Commit message: add visual representation

File: urdf/rover.urdf (robot description, URDF)
Before this commit: robot tracked_rover, 4 links, 3 joints
Links:
- link as_dt1_link: geometry collision box size=0.03 0.03 0.03; visual box size=0.03 0.03 0.03
- link base_link: geometry collision box size=1.18 0.80 0.44; visual box size=1.18 0.80 0.44
- link gps_link: geometry collision cylinder length=0.02 radius=0.04; visual cylinder length=0.02 radius=0.04

Commit message: adding radar module on top

File: urdf/rover.urdf (robot description, URDF)
Before this commit: robot tracked_rover, 4 links, 3 joints
Links:
- added link radar_110_link; collision box size=0.04 0.09 0.13; visual box size=0.004 0.09 0.13
- added link radar_111_link; collision box size=0.04 0.09 0.13; visual box size=0.004 0.09 0.13
- added link radar_112_link; collision box size=0.04 0.09 0.13; visual box size=0.004 0.09 0.13
- added link radar_113_link; collision box size=0.04 0.09 0.13; visual box size=0.004 0.09 0.13
- added link radar_114_link; collision box size=0.04 0.09 0.13; visual box size=0.004 0.09 0.13
- added link radar_115_link; collision box size=0.04 0.09 0.13; visual box size=0.004 0.09 0.13
- added link radar_116_link; collision box size=0.04 0.09 0.13; visual box size=0.004 0.09 0.13
- added link radar_117_link; collision box size=0.04 0.09 0.13; visual box size=0.004 0.09 0.13
- added link radar_118_link; collision box size=0.04 0.09 0.13; visual box size=0.004 0.09 0.13
- added link radar_119_link; collision box size=0.04 0.09 0.13; visual box size=0.004 0.09 0.13
- added link radar_120_link; collision box size=0.04 0.09 0.13; visual box size=0.004 0.09 0.13
- added link radar_121_link; collision box size=0.04 0.09 0.13; visual box size=0.004 0.09 0.13
- added link radar_122_link; collision box size=0.04 0.09 0.13; visual box size=0.004 0.09 0.13
- added link radar_123_link; collision box size=0.04 0.09 0.13; visual box size=0.004 0.09 0.13
- added link radar_124_link; collision box size=0.04 0.09 0.13; visual box size=0.004 0.09 0.13
- added link radar_125_link; collision box size=0.04 0.09 0.13; visual box size=0.004 0.09 0.13
- added link radar_126_link; collision box size=0.04 0.09 0.13; visual box size=0.004 0.09 0.13
- added link radar_127_link; collision box size=0.04 0.09 0.13; visual box size=0.004 0.09 0.13
- added link radar_128_link; collision box size=0.04 0.09 0.13; visual box size=0.004 0.09 0.13
- added link radar_129_link; collision box size=0.04 0.09 0.13; visual box size=0.004 0.09 0.13
- link base_link: geometry collision box size=0.21 0.44 0.04; collision box size=0.24 0.18 0.10
Joints:
- added joint base_to_radar_110_link: type fixed, parent base_link, child radar_110_link, origin xyz=-0.3898470249727761 0.275065749611853 0.56 rpy=0 -0.523599 2.199115
- added joint base_to_radar_111_link: type fixed, parent base_link, child radar_111_link, origin xyz=-0.29506590996827614 0.323359172689655 0.56 rpy=0 -0.523599 1.884956
- added joint base_to_radar_112_link: type fixed, parent base_link, child radar_112_link, origin xyz=-0.18999988888973518 0.3399999999999819 0.56 rpy=0 -0.523599 1.570796
- added joint base_to_radar_113_link: type fixed, parent base_link, child radar_113_link, origin xyz=-0.08493420204664806 0.32335920908553917 0.56 rpy=0 -0.523599 1.256637
- added joint base_to_radar_114_link: type fixed, parent base_link, child radar_114_link, origin xyz=0.009846929687180983 0.2750658188408857 0.56 rpy=0 -0.523599 0.942478
- added joint base_to_radar_115_link: type fixed, parent base_link, child radar_115_link, origin xyz=0.08506568430285044 0.19984711486284873 0.56 rpy=0 -0.523599 0.628319
- added joint base_to_radar_116_link: type fixed, parent base_link, child radar_116_link, origin xyz=0.1333592434204885 0.10506569228120705 0.56 rpy=0 -0.523599 0.314159
- added joint base_to_radar_117_link: type fixed, parent base_link, child radar_117_link, origin xyz=0.15000000000000002 0.0 0.56 rpy=0 -0.523599 0.0
- added joint base_to_radar_118_link: type fixed, parent base_link, child radar_118_link, origin xyz=0.13335921114643734 -0.10506579161056064 0.56 rpy=0 -0.523599 5.969026
- added joint base_to_radar_119_link: type fixed, parent base_link, child radar_119_link, origin xyz=0.08506582276094521 -0.19984692429167955 0.56 rpy=0 -0.523599 5.654867
- added joint base_to_radar_120_link: type fixed, parent base_link, child radar_120_link, origin xyz=0.009847120258347442 -0.27506568038278717 0.56 rpy=0 -0.523599 5.340708
- added joint base_to_radar_121_link: type fixed, parent base_link, child radar_121_link, origin xyz=-0.08493430137600112 -0.32335924135959226 0.56 rpy=0 -0.523599 5.026548
- added joint base_to_radar_122_link: type fixed, parent base_link, child radar_122_link, origin xyz=-0.18999999333079456 -0.33999999999999997 0.56 rpy=0 -0.523599 4.712389
- added joint base_to_radar_123_link: type fixed, parent base_link, child radar_123_link, origin xyz=-0.2950656859384152 -0.32335924548138456 0.56 rpy=0 -0.523599 4.39823
- added joint base_to_radar_124_link: type fixed, parent base_link, child radar_124_link, origin xyz=-0.3898471094673501 -0.27506568822291344 0.56 rpy=0 -0.523599 4.08407
- added joint base_to_radar_125_link: type fixed, parent base_link, child radar_125_link, origin xyz=-0.4650658149208261 -0.1998469350826823 0.56 rpy=0 -0.523599 3.769911
- added joint base_to_radar_126_link: type fixed, parent base_link, child radar_126_link, origin xyz=-0.5133592070246409 -0.10506580429614308 0.56 rpy=0 -0.523599 3.455752
- added joint base_to_radar_127_link: type fixed, parent base_link, child radar_127_link, origin xyz=-0.5299999999999796 -1.177794702505938e-07 0.56 rpy=0 -0.523599 3.141593
- added joint base_to_radar_128_link: type fixed, parent base_link, child radar_128_link, origin xyz=-0.5133591747505554 0.10506590362548561 0.56 rpy=0 -0.523599 2.827433
- added joint base_to_radar_129_link: type fixed, parent base_link, child radar_129_link, origin xyz=-0.4650657535319143 0.19984701957727616 0.56 rpy=0 -0.523599 2.513274
